Commit message: changed the launch parameter from copernicus to volta

File: catkin_world_ws/src/volta_description/urdf/volta.urdf.xacro (robot description, xacro)
@@ -34,10 +34,10 @@
     <xacro:arg name="robot_namespace" default="/" />
     <xacro:arg name="tf_pre" default=""/>
-    <xacro:arg name="lidar_enabled" default="true"/>
-    <xacro:arg name="rplidar_a3_enabled" default="true"/>
+    <xacro:arg name="lidar_enabled" default="false"/>
+    <xacro:arg name="rplidar_a3_enabled" default="false"/>
     <xacro:arg name="hokuyo_ust_10lx_enabled" default="false"/>
     <xacro:arg name="imu_enabled" default="true"/>
-    <xacro:arg name="camera_enabled" default="true"/>
-    <xacro:arg name="intel_d435i_enabled" default="true"/>
+    <xacro:arg name="camera_enabled" default="false"/>
+    <xacro:arg name="intel_d435i_enabled" default="false"/>
     <xacro:arg name="orbbec_astra_pro_enabled" default="false"/>
     <xacro:macro name="volta_robot">
@@ -111,4 +111,8 @@
             <xacro:camera_ intel_d435i_enabled="$(arg intel_d435i_enabled)" orbbec_astra_pro_enabled="$(arg orbbec_astra_pro_enabled)" robot_namespace="$(arg robot_namespace)"></xacro:camera_>
         </xacro:if>
+        <xacro:include filename="$(find velodyne_description)/urdf/VLP-16.urdf.xacro"/>
+        <xacro:VLP-16 parent="base_link" name="velodyne" topic="/velodyne_points" hz="10" samples="360" gpu="false" min_angle="-1.57" max_angle="1.57" min_range="0.1">
+            <origin xyz="0.125 0 0.2" rpy="0 0 0" />
+        </xacro:VLP-16>
         <!-- Robot Gazebo tag -->
         <gazebo>

Commit message: fixed the lidar placement

File: catkin_world_ws/src/volta_description/urdf/volta.urdf.xacro (robot description, xacro)
@@ -113,5 +113,5 @@
         <xacro:include filename="$(find velodyne_description)/urdf/VLP-16.urdf.xacro"/>
         <xacro:VLP-16 parent="base_link" name="velodyne" topic="/velodyne_points" hz="10" samples="360" gpu="false" min_angle="-1.57" max_angle="1.57" min_range="0.1">
-            <origin xyz="0.125 0 0.2" rpy="0 0 0" />
+            <origin xyz="0.206 0 0.115" rpy="0 0 0" />
         </xacro:VLP-16>
         <!-- Robot Gazebo tag -->
